Commit message: Modify the urdf model

File: catkin_ws/src/hardware/autobot_description/urdf/autobot_urdf.urdf (robot description, URDF)
Before this commit: robot autobot, 4 links, 3 joints
Links:
- removed link front_l_wheel
- added link front_l_wheel_link; visual cylinder length=0.055 radius=0.065
- added link front_r_wheel_link; visual cylinder length=0.055 radius=0.065
Joints:
- added joint front_l_r_wheel_joint: type fixed, parent front_l_wheel_link, child front_r_wheel_link, origin xyz=0 -0.215 0 rpy=0 0 0
- joint drive_front_l_wheel_joint: child front_l_wheel -> front_l_wheel_link

Commit message: modify the urdf file to move the two wheels

File: catkin_ws/src/hardware/autobot_description/urdf/autobot_urdf.urdf (robot description, URDF)
Before this commit: robot autobot, 5 links, 4 joints
Links:
- removed link drive_front_l_link
- removed link front_l_wheel_link
- removed link front_r_wheel_link
- added link steer_front_r_link; visual cylinder length=0.005 radius=0.005
Joints:
- removed joint drive_front_l_joint
- removed joint drive_front_l_wheel_joint
- removed joint front_l_r_wheel_joint
- added joint steer_front_r_joint: type revolute, parent base_link, child steer_front_r_link, origin xyz=0.14 -0.135 0 rpy=0 0 0, axis 0 0 1, limit lower=-0.2 upper=0.2 effort=0.1 velocity=0.005
